File: schema/Untitled/Untitled.kicad_pcb (KiCad board)
At the start: 2 copper layers, 27 parts, among them J1 batteries 2x aa, SW1 SW_Push, SW2 SW_Push, U1 ATtiny84A-P, U2 74HC595, U3 74HC595, U4 CC56-12SURKWA

Commit message: THC
Parts:
- C1: footprint Capacitor_THT:CP_Radial_D8.0mm_P3.80mm -> Capacitor_THT:CP_Radial_D5.0mm_P2.50mm
- SW1, SW2: footprint Button_Switch_SMD:SW_Push_1P1T_NO_CK_PTS125Sx43SMTR -> Button_Switch_SMD:SW_SPST_Omron_B3FS-101xP
- moved TP1 117.5 mm to (135.4, 157.5)
- moved TP4 112.2 mm to (131.9, 155.1)
- moved TP6 111.7 mm to (138.1, 164.2)
- moved TP5 105.9 mm to (133.6, 166.3)
- moved H2 103.6 mm to (144.0, 116.8)
- moved TP2 98.2 mm to (113.9, 157.4)
- moved TP3 96.0 mm to (114.2, 149.9)
- moved SW2 83.2 mm to (140.2, 147.9), turned to -90 degrees
- moved J1 72.2 mm to (104.6, 166.8)
- moved C2 70.7 mm to (109.2, 166.8), turned to 90 degrees
- moved C1 62.2 mm to (124.6, 166.4), turned to 90 degrees
- moved H1 61.4 mm to (100.3, 116.8)
- moved SW1 47.4 mm to (104.0, 147.9), turned to 90 degrees
- moved R2 2.34 mm to (147.1, 124.0)
Connections:
- SW1 pad 2: Net-(U1-XTAL1/PB0) -> Net-(U1-PA7)
- SW2 pad 2: Net-(U1-PA1) -> Net-(U1-PA3)
- U1 pad 10: /s_latch -> Net-(U1-PA3)
- U1 pad 11: unconnected-(U1-PA2-Pad11) -> /s_data
- U1 pad 12: Net-(U1-PA1) -> /s_clock
- U1 pad 13: unconnected-(U1-AREF/PA0-Pad13) -> /s_clear
- U1 pad 2: Net-(U1-XTAL1/PB0) -> /s_latch
- U1 pad 3: /s_data -> unconnected-(U1-XTAL2/PB1-Pad3)
- U1 pad 5: /s_clock -> unconnected-(U1-PB2-Pad5)
- U1 pad 6: /s_clear -> Net-(U1-PA7)
Routing:
- net VCC: track 39.0 -> 147.6 mm
- net GND: track 63.9 -> 166.8 mm, vias 0 -> 2
- net /s_clock: track 0.00 -> 51.4 mm, vias 0 -> 2
- net /s_clear: track 0.00 -> 43.9 mm, vias 0 -> 2
- net /s_latch: track 0.00 -> 43.9 mm
- net /s_data: track 0.00 -> 28.4 mm
- net Net-(U2-QH'): track 0.00 -> 18.9 mm
- net Net-(U1-PA7): track 0.00 -> 14.7 mm
- net Net-(U1-PA3): track 0.00 -> 8.93 mm
- net /miso: track 0.00 -> 8.13 mm
- net /mosi: track 0.00 -> 5.77 mm
- net /reset: track 0.00 -> 5.47 mm
- net Net-(U4-b): track 37.3 -> 41.3 mm
- net /sck: track 0.00 -> 2.67 mm
- net /b: track 7.25 -> 4.97 mm
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
Commit message: ultimos toques a la pcb
Parts:
- removed H3, H4: MountingHole, MountingHole:MountingHole_3.2mm_M3
- U1: footprint Package_DIP:DIP-14_W7.62mm -> Package_DIP:DIP-14_W7.62mm_SMDSocket_SmallPads
- U2, U3: footprint Package_DIP:DIP-16_W7.62mm_LongPads -> Package_DIP:DIP-16_W7.62mm_SMDSocket_SmallPads
- moved U2 56.0 mm to (91.9, 117.6)
- moved U3 56.0 mm to (63.8, 117.6)
- moved TP6 48.6 mm to (92.2, 148.6)
- moved H2 48.4 mm to (98.0, 101.6)
- moved R1 48.4 mm to (61.2, 106.7)
- moved SW1 48.4 mm to (58.0, 132.6)
- moved SW2 48.4 mm to (94.3, 132.6)
- moved TP3 48.4 mm to (68.2, 134.7)
- moved C2 48.4 mm to (63.2, 151.5)
- moved H1 48.4 mm to (54.4, 101.6)
- moved R2 48.4 mm to (101.1, 108.7)
- moved R3 48.4 mm to (79.4, 106.7)
- moved R4 48.4 mm to (72.0, 106.7)
- moved R5 48.4 mm to (68.1, 106.7)
- moved R7 48.4 mm to (83.1, 106.7)
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Other:
- board outline added: 55.9 x 82.6 mm
- board text added: "+"
- board text added: "-"
- board text added: "Ticker"
- board text added: "ck"
- board text added: "gnd"
- board text added: "miso"
- board text added: "mosi"
- board text added: "rst"

Commit message: pcb que se realizará
Routing:
- net /s_clock: track 51.4 -> 53.4 mm
- net /s_clear: track 43.9 -> 45.8 mm
- net GND: track 166.8 -> 166.0 mm
Other:
- board text added: "s_clear"
- board text added: "s_clk"
Changed lines of the file:
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@@
 		(net 10)
+	)
+	(gr_circle
+		(center 56.642 125.476)
+		(end 55.88 125.476)
+		(stroke
+			(width 1.55)
+			(type default)
+		)
+		(fill no)
+		(layer "B.Cu")
+		(net 18)
+	)
+	(gr_circle
+		(center 87.884 132.08)
+		(end 88.392 131.826)
+		(stroke
+			(width 1.55)
+			(type default)
+		)
+		(fill no)
+		(layer "B.Cu")
+		(net 19)
+	)
+	(gr_circle
+		(center 60.706 125.476)
+		(end 61.468 125.476)
+		(stroke
+			(width 1.55)
+			(type default)
+		)
+		(fill no)
+		(layer "B.Cu")
+		(net 19)
+	)
+	(gr_circle
+		(center 78.74 122.428)
+		(end 79.502 122.936)
+		(stroke
+			(width 1.55)
+			(type default)
+		)
+		(fill no)
+		(layer "B.Cu")
+		(net 1)
+	)
+	(gr_circle
+		(center 67.31 126.746)
+		(end 68.072 126.492)
+		(stroke
+			(width 1.55)
+			(type default)
+		)
+		(fill no)
+		(layer "B.Cu")
+		(net 1)
+	)
+	(gr_circle
+		(center 86.106 129.54)
+		(end 86.36 129.286)
+		(stroke
+			(width 1.55)
+			(type default)
+		)
+		(fill no)
+		(layer "B.Cu")
+		(net 18)
+	)
+	(gr_line
+		(start 76.2 97.282)
+		(end 76.2 115.316)
+		(stroke
+			(width 0.55)
+			(type dash_dot_dot)
+		)
+		(layer "B.Cu")
+	)
+	(gr_line
+		(start 66.04 101.6)
+		(end 86.36 101.6)
+		(stroke
+			(width 0.2)
+			(type dash)
+		)
+		(layer "B.Cu")
 	)
 	(gr_rect
@@
 		)
 	)
+	(gr_text "s_clk"
+		(at 87.122 126.746 0)
+		(layer "B.Cu")
+		(effects
+			(font
+				(size 1.5 1.5)
+				(thickness 0.3)
+				(bold yes)
+			)
+			(justify left bottom mirror)
+		)
+	)
+	(gr_text "gnd"
+		(at 73.66 124.46 0)
+		(layer "B.Cu")
+		(effects
+			(font
+				(size 1.5 1.5)
+				(thickness 0.3)
+				(bold yes)
+			)
+			(justify left bottom mirror)
+		)
+	)
+	(gr_text "s_clear"
+		(at 73.914 133.096 0)
+		(layer "B.Cu")
+		(effects
+			(font
+				(size 1.5 1.5)
+				(thickness 0.3)
+				(bold yes)
+			)
+			(justify left bottom mirror)
+		)
+	)
 	(segment
 		(start 80.264 116.586)
@@
 	)
 	(segment
+		(start 54.864 149.352)
+		(end 55.372 148.844)
+		(width 0.38)
+		(layer "F.Cu")
+		(net 1)
+	)
+	(segment
 		(start 65.024 117.094)
 		(end 55.626 117.094)
@@
 	)
 	(segment
+		(start 55.372 148.844)
+		(end 60.9238 148.844)
+		(width 0.38)
+		(layer "F.Cu")
+		(net 1)
+	)
+	(segment
 		(start 62.8904 145.6944)
 		(end 55.726 138.53)
@@
 	)
 	(segment
+		(start 60.9238 148.844)
+		(end 63.2206 146.5472)
+		(width 0.38)
+		(layer "F.Cu")
+		(net 1)
+	)
+	(segment
 		(start 54.864 116.078)
 		(end 54.864 113.792)
@@
 	)
 	(segment
-		(start 60.0124 146.5472)
-		(end 63.2206 146.5472)
-		(width 0.38)
-		(layer "F.Cu")
-		(net 1)
-	)
-	(segment
 		(start 65.532 116.586)
 		(end 65.024 117.094)
@@
 		(start 53.694 128.624)
 		(end 55.726 128.624)
-		(width 0.38)
-		(layer "F.Cu")
-		(net 1)
-	)
-	(segment
-		(start 54.9978 151.5618)
-		(end 60.0124 146.5472)
 		(width 0.38)
 		(layer "F.Cu")
@@
 	)
 	(segment
-		(start 62.729 130.801)
+		(start 57.404 128.778)
 		(end 57.404 125.476)
+		(width 0.38)
+		(layer "B.Cu")
+		(net 18)
+	)
+	(segment
+		(start 59.427 130.801)
+		(end 57.404 128.778)
+		(width 0.38)
+		(layer "B.Cu")
+		(net 18)
+	)
+	(segment
+		(start 84.845 130.801)
+		(end 59.427 130.801)
 		(width 0.38)
 		(layer "B.Cu")
@@
 	)
 	(segment
-		(start 84.845 130.801)
-		(end 62.729 130.801)
-		(width 0.38)
-		(layer "B.Cu")
-		(net 18)
-	)
-	(segment
 		(start 88.138 129.794)
 		(end 88.138 123.698)
@@
 	)
 	(segment
-		(start 59.944 121.768677)
-		(end 59.944 125.73)
-		(width 0.38)
-		(layer "F.Cu")
-		(net 19)
-	)
-	(segment
 		(start 83.312 132.08)
 		(end 85.852 132.08)
@@
 	)
 	(segment
+		(start 59.944 121.768677)
+		(end 59.944 125.222)
+		(width 0.38)
+		(layer "F.Cu")
+		(net 19)
+	)
+	(segment
 		(start 85.852 132.08)
 		(end 87.884 132.08)
@@
 		(net 19)
 	)
+	(segment
+		(start 59.944 125.222)
+		(end 60.452 125.73)
+		(width 0.38)
+		(layer "F.Cu")
+		(net 19)
+	)
 	(via
-		(at 59.944 125.73)
+		(at 60.452 125.73)
 		(size 1.5)
 		(drill 0.8)
@@
 	)
 	(segment
-		(start 86.407192 128.27)
-		(end 62.484 128.27)
-		(width 0.38)
-		(layer "B.Cu")
-		(net 19)
-	)
-	(segment
-		(start 62.484 128.27)
-		(end 59.944 125.73)
-		(width 0.38)
-		(layer "B.Cu")
-		(net 19)
-	)
-	(segment
-		(start 87.884 132.08)
-		(end 87.884 129.746808)
-		(width 0.38)
-		(layer "B.Cu")
-		(net 19)
-	)
-	(segment
-		(start 87.884 129.746808)
-		(end 86.407192 128.27)
-		(width 0.38)
-		(layer "B.Cu")
+		(start 86.868 127.508)
+		(end 87.884 128.524)
+		(width 0.38)
+		(layer "B.Cu")
+		(net 19)
+	)
+	(segment
+		(start 87.884 128.524)
+		(end 87.884 132.08)
+		(width 0.38)
+		(layer "B.Cu")
+		(net 19)
+	)
+	(segment
+		(start 60.452 125.73)
+		(end 60.452 126.238)
+		(width 0.38)
+		(layer "B.Cu")
+		(net 19)
+	)
+	(segment
+		(start 60.452 126.238)
+		(end 63.246 129.032)
+		(width 0.38)
+		(layer "B.Cu")
+		(net 19)
+	)
+	(segment
+		(start 71.628 127.508)
+		(end 86.868 127.508)
+		(width 0.38)
+		(layer "B.Cu")
+		(net 19)
+	)
+	(segment
+		(start 70.104 129.032)
+		(end 71.628 127.508)
+		(width 0.38)
+		(layer "B.Cu")
+		(net 19)
+	)
+	(segment
+		(start 63.246 129.032)
+		(end 70.104 129.032)
+		(width 0.38)
+		(layer "B.Cu")
